File: ColorSensingLEDStrip.kicad_pcb (KiCad board)
At the start: 2 copper layers, 99.1 x 68.6 mm, 14 parts, among them J1 Barrel_Jack_Switch, J2 4-Wire Screw Terminal, SW1 Rotary_Encoder_Switch, U1 Adafruit_AS7341, U2 OLED

Commit message: v2.0 PCB files
Parts:
- moved U2 35.7 mm to (123.5, 98.4)
- moved A1 23.6 mm to (135.9, 75.6)
- moved U1 23.6 mm to (157.5, 87.0)
- moved REF** 23.6 mm to (185.4, 67.9)
- moved REF** 23.6 mm to (185.4, 126.4)
- moved C2 23.6 mm to (108.0, 121.3)
- moved J1 23.6 mm to (103.5, 109.2)
- moved REF** 23.6 mm to (96.5, 67.9)
- moved C1 23.6 mm to (111.8, 126.4)
- moved REF** 23.6 mm to (96.5, 126.4)
- moved C4 23.6 mm to (177.8, 70.5)
- moved SW1 23.6 mm to (176.5, 106.0)
- moved C3 23.6 mm to (184.2, 76.8)
- moved J2 23.6 mm to (184.2, 85.7)
Routing:
- net +5V: track 264.3 -> 258.7 mm
- net I2C_SDA: track 61.9 -> 58.6 mm
- net I2C_SCL: track 55.3 -> 51.9 mm
Other:
- board text added: "Color Sensing LED Strip V2.0 - Sabrina Pereira & Co."
- board text removed: "Color Sensing LED Strip V1.0 - Sabrina Pereira & Co."
